File: Hardware/yrdy/echelon/echelon.kicad_pcb (KiCad board)
At the start: 2 copper layers, 3 parts, among them U1 ADC081C021CIMM, U2 ATxmega384D3-A, U4 ESP8266EX

Commit message: kkk
Other:
- board text added: "Component Pcb for Utility"
Changed lines of the file:
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@@
     )
   )
+  (gr_text "Component Pcb for Utility\n" (at 180.34 170.18) (layer "F.Cu")
+    (effects (font (size 1.5 1.5) (thickness 0.3) bold) (justify left bottom))
+  )
+  (gr_text_box "microcontroller\n"
+    (start 119.38 99.06) (end 127 104.14) (layer "F.Cu")
+      (effects (font (size 1.5 1.5) (thickness 0.3) bold) (justify left top))
+    (stroke (width 0.2) (type solid))  )
+  (gr_text_box "wifi\n"
+    (start 144.78 91.44) (end 160.02 93.98) (layer "F.Cu")
+      (effects (font (size 1.5 1.5) (thickness 0.3) bold) (justify left top))
+    (stroke (width 0.2) (type solid))  )
+  (gr_text_box "bluetooth\n"
+    (start 144.78 81.28) (end 157.48 83.82) (layer "F.Cu")
+      (effects (font (size 1.5 1.5) (thickness 0.3) bold) (justify left top))
+    (stroke (width 0.2) (type solid))  )
 )

Commit message: d
Parts:
- added U5: ATxmega384D3-A, Package_QFP:TQFP-64_14x14mm_P0.8mm, F.Cu at (126.9, 67.7)
- added U6: FU540-C000, Package_BGA:BGA-484_23.0x23.0mm_Layout22x22_P1.0mm, F.Cu at (70.6, 50.3)

Commit message: l
Parts:
- added U5: FE310-G002, Package_DFN_QFN:QFN-48-1EP_6x6mm_P0.4mm_EP4.2x4.2mm_ThermalVias, F.Cu at (88.5, 58.8)
Connections:
- U4 pad 33: unconnected-(U4-GND-Pad33) -> GND
- U6 pad A12: unconnected-(U6C-GEMGXL_0_RXD_0-PadA12) -> Net-(U6C-GEMGXL_0_RXD_0)
- U6 pad A19: unconnected-(U6E-MSEL_MSEL_0-PadA19) -> Net-(U6E-MSEL_MSEL_0)
- U6 pad A8: unconnected-(U6C-GEMGXL_0_RXD_5-PadA8) -> Net-(U6C-GEMGXL_0_RXD_0)
- U6 pad AA11: unconnected-(U6B-DDR_MEM_D[63]-PadAA11) -> Net-(U6B-DDR_MEM_D[56])
- U6 pad AA13: unconnected-(U6B-DDR_MEM_D[56]-PadAA13) -> Net-(U6B-DDR_MEM_D[56])
- U6 pad AA4: Net-(U6B-DDR_MEM_DM[5]) -> Net-(U6B-DDR_MEM_D[40])
- U6 pad B1: Net-(U6B-DDR_MEM_DM[0]) -> unconnected-(U6B-DDR_MEM_D[1]-PadB1)
- U6 pad B12: unconnected-(U6C-GEMGXL_0_TXD_0-PadB12) -> Net-(U6C-GEMGXL_0_TXD_0)
- U6 pad B19: unconnected-(U6E-MSEL_MSEL_3-PadB19) -> Net-(U6E-MSEL_MSEL_0)
- U6 pad B4: unconnected-(U6B-DDR_MEM_D[16]-PadB4) -> Net-(U6B-DDR_MEM_D[16])
- U6 pad B6: Net-(U6B-DDR_MEM_DM[2]) -> Net-(U6B-DDR_MEM_D[16])
- U6 pad C1: unconnected-(U6B-DDR_MEM_D[4]-PadC1) -> Net-(U6B-DDR_MEM_D[0])
- U6 pad C10: unconnected-(U6C-GEMGXL_0_TXD_4-PadC10) -> Net-(U6C-GEMGXL_0_TXD_0)
- U6 pad C14: unconnected-(U6E-PRCI_RSVD15-PadC14) -> Net-(U6E-PRCI_RSVD13)
- U6 pad C20: unconnected-(U6D-GPIO_0_P_7-PadC20) -> Net-(U6D-GPIO_0_P_0)
- U6 pad C3: unconnected-(U6B-DDR_MEM_D[27]-PadC3) -> Net-(U6B-DDR_MEM_D[24])
- U6 pad C4: unconnected-(U6B-DDR_MEM_D[24]-PadC4) -> Net-(U6B-DDR_MEM_D[24])
- U6 pad C6: Net-(U6B-DDR_MEM_DM[2]) -> unconnected-(U6B-DDR_MEM_DM[2]-PadC6)
- U6 pad C7: Net-(U6B-DDR_MEM_DM[3]) -> Net-(U6B-DDR_MEM_D[24])
- U6 pad C9: unconnected-(U6C-GEMGXL_0_RXD_6-PadC9) -> Net-(U6C-GEMGXL_0_RXD_0)
- U6 pad D16: unconnected-(U6E-PRCI_RSVD3-PadD16) -> Net-(U6E-PRCI_RSVD3)
- U6 pad D17: unconnected-(U6E-PRCI_RSVD10-PadD17) -> Net-(U6E-PRCI_RSVD10)
- U6 pad D2: unconnected-(U6B-DDR_MEM_D[0]-PadD2) -> Net-(U6B-DDR_MEM_D[0])
- U6 pad D5: Net-(U6B-DDR_MEM_DM[3]) -> unconnected-(U6B-DDR_MEM_DM[3]-PadD5)
- U6 pad D6: Net-(U6B-DDR_MEM_DM[3]) -> unconnected-(U6B-DDR_MEM_D[26]-PadD6)
- U6 pad D8: unconnected-(U6B-DDR_RSVD1-PadD8) -> Net-(U6B-DDR_RSVD0)
- U6 pad D9: unconnected-(U6C-GEMGXL_0_TXD_7-PadD9) -> Net-(U6C-GEMGXL_0_TXD_0)
- U6 pad E14: unconnected-(U6E-PRCI_RSVD12-PadE14) -> Net-(U6E-PRCI_RSVD10)
- U6 pad E16: unconnected-(U6E-PRCI_RSVD9-PadE16) -> Net-(U6E-PRCI_RSVD3)
- U6 pad E2: Net-(U6B-DDR_MEM_DM[0]) -> Net-(U6B-DDR_MEM_D[0])
- U6 pad E5: Net-(U6B-DDR_MEM_DM[0]) -> unconnected-(U6B-DDR_MEM_DM[0]-PadE5)
- U6 pad E6: unconnected-(U6B-DDR_MEM_D[28]-PadE6) -> Net-(U6B-DDR_MEM_D[24])
- U6 pad E8: unconnected-(U6B-DDR_RSVD0-PadE8) -> Net-(U6B-DDR_RSVD0)
- U6 pad E9: unconnected-(U6C-GEMGXL_0_RXD_7-PadE9) -> Net-(U6C-GEMGXL_0_RXD_0)
- U6 pad F14: unconnected-(U6E-PRCI_RSVD13-PadF14) -> Net-(U6E-PRCI_RSVD13)
- U6 pad F17: unconnected-(U6D-GPIO_0_P_0-PadF17) -> Net-(U6D-GPIO_0_P_0)
- U6 pad F19: unconnected-(U6D-PWM_1_P_3-PadF19) -> Net-(U6D-PWM_0_P_0)
- U6 pad F4: Net-(U6B-DDR_MEM_DM[0]) -> unconnected-(U6B-DDR_MEM_D[2]-PadF4)
- U6 pad F5: Net-(U6B-DDR_MEM_DM[1]) -> Net-(U6B-DDR_MEM_D[10])
- U6 pad F9: unconnected-(U6B-DDR_RSVD3-PadF9) -> Net-(U6B-DDR_RSVD0)
- U6 pad G17: unconnected-(U6D-GPIO_0_P_15-PadG17) -> Net-(U6D-GPIO_0_P_0)
- U6 pad G19: unconnected-(U6D-PWM_0_P_0-PadG19) -> Net-(U6D-PWM_0_P_0)
- U6 pad G20: unconnected-(U6D-PWM_0_P_3-PadG20) -> Net-(U6D-PWM_0_P_0)
- U6 pad G22: unconnected-(U6D-QSPI_1_DQ_0-PadG22) -> Net-(U6D-QSPI_1_DQ_0)
- U6 pad G3: Net-(U6B-DDR_MEM_DM[0]) -> Net-(U6B-DDR_MEM_D[0])
- U6 pad G5: Net-(U6B-DDR_MEM_DM[1]) -> unconnected-(U6B-DDR_MEM_DM[1]-PadG5)
- U6 pad H19: unconnected-(U6D-QSPI_1_CS_2-PadH19) -> Net-(U6D-QSPI_1_CS_0)
- U6 pad H20: unconnected-(U6D-QSPI_0_DQ_3-PadH20) -> Net-(U6D-QSPI_0_DQ_0)
- U6 pad H21: unconnected-(U6D-QSPI_0_DQ_0-PadH21) -> Net-(U6D-QSPI_0_DQ_0)
- U6 pad H4: unconnected-(U6B-DDR_MEM_D[8]-PadH4) -> Net-(U6B-DDR_MEM_D[10])
- U6 pad J17: unconnected-(U6D-QSPI_1_DQ_3-PadJ17) -> Net-(U6D-QSPI_1_DQ_0)
- U6 pad J18: unconnected-(U6D-QSPI_1_DQ_1-PadJ18) -> Net-(U6D-QSPI_1_DQ_0)
- U6 pad J20: unconnected-(U6D-QSPI_1_CS_3-PadJ20) -> Net-(U6D-QSPI_1_CS_0)
- U6 pad J4: Net-(U6B-DDR_MEM_DM[1]) -> Net-(U6B-DDR_MEM_D[10])
- U6 pad J5: unconnected-(U6B-DDR_MEM_ECC_DM-PadJ5) -> Net-(U6B-DDR_MEM_ECC_DM)
- U6 pad K17: unconnected-(U6D-QSPI_1_CS_0-PadK17) -> Net-(U6D-QSPI_1_CS_0)
- U6 pad K5: unconnected-(U6B-DDR_MEM_CLK-PadK5) -> Net-(U6B-DDR_MEM_CLK)
- U6 pad L17: unconnected-(U6A-CL_0_C2B_D_31-PadL17) -> Net-(U6A-CL_0_C2B_D_0)
- U6 pad L3: unconnected-(U6B-DDR_MEM_ECC_D[7]-PadL3) -> Net-(U6B-DDR_MEM_ECC_DM)
- U6 pad L5: unconnected-(U6B-DDR_MEM_CLK_N-PadL5) -> Net-(U6B-DDR_MEM_CLK)
- U6 pad M17: unconnected-(U6A-CL_0_C2B_D_15-PadM17) -> Net-(U6A-CL_0_C2B_D_0)
- U6 pad M4: unconnected-(U6B-DDR_MEM_BANK[0]-PadM4) -> Net-(U6B-DDR_MEM_ADDR[15])
- U6 pad M5: unconnected-(U6B-DDR_MEM_BANK[2]-PadM5) -> Net-(U6B-DDR_MEM_ADDR[15])
- U6 pad T19: unconnected-(U6A-CL_0_C2B_D_0-PadT19) -> Net-(U6A-CL_0_C2B_D_0)
- U6 pad U3: Net-(U6B-DDR_MEM_ADDR[14]) -> unconnected-(U6B-DDR_MEM_ADDR[14]-PadU3)
- U6 pad V19: unconnected-(U6A-CL_0_B2C_D_15-PadV19) -> Net-(U6A-CL_0_B2C_D_0)
- U6 pad V3: Net-(U6B-DDR_MEM_ADDR[14]) -> Net-(U6B-DDR_MEM_ADDR[15])
- U6 pad V5: unconnected-(U6B-DDR_MEM_D[40]-PadV5) -> Net-(U6B-DDR_MEM_D[40])
- U6 pad W10: Net-(U6B-DDR_MEM_DM[6]) -> unconnected-(U6B-DDR_MEM_DM[6]-PadW10)
- U6 pad W5: Net-(U6B-DDR_MEM_DM[5]) -> unconnected-(U6B-DDR_MEM_DM[5]-PadW5)
- U6 pad W8: Net-(U6B-DDR_MEM_DM[6]) -> Net-(U6B-DDR_MEM_D[48])
- U6 pad W9: Net-(U6B-DDR_MEM_DM[6]) -> Net-(U6B-DDR_MEM_D[48])
- U6 pad Y12: unconnected-(U6B-DDR_MEM_D[48]-PadY12) -> Net-(U6B-DDR_MEM_D[48])
- U6 pad Y16: unconnected-(U6A-CL_0_B2C_D_0-PadY16) -> Net-(U6A-CL_0_B2C_D_0)
- U6 pad Y21: unconnected-(U6A-CL_0_B2C_D_31-PadY21) -> Net-(U6A-CL_0_B2C_D_0)
- U6 pad Y3: Net-(U6B-DDR_MEM_DM[5]) -> Net-(U6B-DDR_MEM_D[40])
- U6 pad Y5: Net-(U6B-DDR_MEM_ADDR[14]) -> unconnected-(U6B-DDR_MEM_RESET_N-PadY5)
