File: Hardware/yrdy/echelon/motherboard.kicad_sch (KiCad schematic)
At the start: 0 parts

Commit message: d
Parts:
- added U6: FU540-C000, Package_BGA:BGA-484_23.0x23.0mm_Layout22x22_P1.0mm, symbol MCU_SiFive:FU540-C000
Connections:
- new net: U6.A1 (VSS), U6.A14 (VSS), U6.A18 (VSS), U6.A2 (VSS), U6.A22 (VSS), U6.A3 (VSS), U6.A9 (VSS), U6.AA2 (VSS), U6.AB1 (VSS), U6.AB10 (VSS), U6.AB13 (VSS), U6.AB17 (VSS), U6.AB22 (VSS), U6.AB4 (VSS), U6.AB7 (VSS), U6.D1 (VSS), U6.D12 (VSS), U6.E22 (VSS), U6.E4 (VSS), U6.F7 (VSS), U6.G10 (VSS), U6.G12 (VSS), U6.G16 (VSS), U6.G2 (VSS), U6.G6 (VSS), U6.G8 (VSS), U6.H15 (VSS), U6.H7 (VSS), U6.H9 (VSS), U6.J1 (VSS), U6.J10 (VSS), U6.J16 (VSS), U6.J22 (VSS), U6.J6 (VSS), U6.J8 (VSS), U6.K11 (VSS), U6.K7 (VSS), U6.K9 (VSS), U6.L10 (VSS), U6.L12 (VSS), U6.L14 (VSS), U6.L6 (VSS), U6.L8 (VSS), U6.M11 (VSS), U6.M13 (VSS), U6.M7 (VSS), U6.N10 (VSS), U6.N12 (VSS), U6.N14 (VSS), U6.N6 (VSS), U6.N8 (VSS), U6.P1 (VSS), U6.P11 (VSS), U6.P13 (VSS), U6.P15 (VSS), U6.P22 (VSS), U6.P7 (VSS), U6.P9 (VSS), U6.R10 (VSS), U6.R12 (VSS), U6.R14 (VSS), U6.R16 (VSS), U6.R6 (VSS), U6.R8 (VSS), U6.T11 (VSS), U6.T13 (VSS), U6.T15 (VSS), U6.T17 (VSS), U6.T7 (VSS), U6.T9 (VSS), U6.U10 (VSS), U6.U12 (VSS), U6.U14 (VSS), U6.U16 (VSS), U6.U6 (VSS), U6.U8 (VSS), U6.V1 (VSS), U6.V11 (VSS), U6.V13 (VSS), U6.V15 (VSS), U6.V22 (VSS), U6.V7 (VSS), U6.V9 (VSS)
- new net: U6.AA17 (VDD), U6.B14 (VDD), U6.B18 (VDD), U6.B9 (VDD), U6.E21 (VDD), U6.E3 (VDD), U6.G11 (VDD), U6.G15 (VDD), U6.G9 (VDD), U6.H10 (VDD), U6.H12 (VDD), U6.H14 (VDD), U6.H16 (VDD), U6.H8 (VDD), U6.J15 (VDD), U6.J9 (VDD), U6.K10 (VDD), U6.K21 (VDD), U6.K8 (VDD), U6.L11 (VDD), U6.L13 (VDD), U6.M10 (VDD), U6.M12 (VDD), U6.M14 (VDD), U6.M8 (VDD), U6.N11 (VDD), U6.N13 (VDD), U6.N9 (VDD), U6.P10 (VDD), U6.P12 (VDD), U6.P14 (VDD), U6.P16 (VDD), U6.P2 (VDD), U6.P21 (VDD), U6.P8 (VDD), U6.R11 (VDD), U6.R13 (VDD), U6.R15 (VDD), U6.R9 (VDD), U6.T10 (VDD), U6.T12 (VDD), U6.T14 (VDD), U6.T16 (VDD), U6.T8 (VDD), U6.U11 (VDD), U6.U13 (VDD), U6.U15 (VDD), U6.U9 (VDD), U6.V10 (VDD), U6.V12 (VDD), U6.V14 (VDD), U6.V21 (VDD), U6.V6 (VDD), U6.V8 (VDD)
- new net: U6.G7 (DDR_VDDQ), U6.H6 (DDR_VDDQ), U6.J7 (DDR_VDDQ), U6.K6 (DDR_VDDQ), U6.L7 (DDR_VDDQ), U6.M6 (DDR_VDDQ), U6.N7 (DDR_VDDQ), U6.P6 (DDR_VDDQ), U6.R7 (DDR_VDDQ), U6.T6 (DDR_VDDQ)
- new net: U6.K15 (IVSS), U6.L15 (IVSS), U6.M15 (IVSS), U6.N15 (IVSS)
- new net: U6.K16 (IVDD), U6.L16 (IVDD), U6.M16 (IVDD), U6.N16 (IVDD)
- new net: U6.L9 (DDR_VDDPLL), U6.M9 (DDR_VDDPLL)

Commit message: l
Parts:
- added R1: R, symbol Device:R
